File: Glove.kicad_sch (KiCad schematic)
At the start: 33 parts, among them J1 USB_C_Receptacle_USB2.0, J2 Joystick, Q1 2N7002, Q2 2N7002, U1 LM1117-3.3, U2 ESP32-WROOM-32D, U3 CP2102N-Axx-xQFN24

Commit message: Switch to QFN28 version of CP2102
Signed-off-by: Kozova1 <mug66kk@gmail.com>
Parts:
- removed U3: CP2102N-Axx-xQFN24, Package_DFN_QFN:QFN-24-1EP_4x4mm_P0.5mm_EP2.6x2.6mm, symbol Interface_USB:CP2102N-Axx-xQFN24
- added U3: (no value), symbol Interface_USB:CP2102N-Axx-xQFN28
- BTN_A1: value Button A -> (none); footprint Connector_JST:JST_XH_B2B-XH-A_1x02_P2.50mm_Vertical -> (none)
- BTN_B1: value Button B -> (none); footprint Connector_JST:JST_XH_B2B-XH-A_1x02_P2.50mm_Vertical -> (none)
- BTN_Grab1: value Grab -> (none); footprint Connector_JST:JST_XH_B2B-XH-A_1x02_P2.50mm_Vertical -> (none)
- BTN_Pinch1: value Pinch -> (none); footprint Connector_JST:JST_XH_B2B-XH-A_1x02_P2.50mm_Vertical -> (none)
- BTN_Trigger1: value Trigger -> (none); footprint Connector_JST:JST_XH_B2B-XH-A_1x02_P2.50mm_Vertical -> (none)
- C1, C4, C_In1, C_Out1: value 10uF -> (none); footprint Capacitor_SMD:C_0805_2012Metric_Pad1.18x1.45mm_HandSolder -> (none); LCSC (none) -> C440198
- C2, C3, C5: value 0.1uF -> (none); footprint Capacitor_SMD:C_0805_2012Metric_Pad1.18x1.45mm_HandSolder -> (none); LCSC (none) -> C28233
- C6: value 4.7uF -> (none); footprint Capacitor_SMD:C_0805_2012Metric_Pad1.18x1.45mm_HandSolder -> (none); LCSC (none) -> C1779
- F1: value 3.5A -> (none); footprint Fuse:Fuse_1812_4532Metric_Pad1.30x3.40mm_HandSolder -> (none); LCSC (none) -> C55996
- J1: value USB_C_Receptacle_USB2.0 -> (none); footprint Connector_USB:USB_C_Receptacle_XKB_U262-16XN-4BVC11 -> (none); LCSC (none) -> C319148
- J2: value Joystick -> (none); footprint Connector_JST:JST_XH_B5B-XH-A_1x05_P2.50mm_Vertical -> (none)
- Q1, Q2: value 2N7002 -> (none); footprint Package_TO_SOT_SMD:SOT-23 -> (none); LCSC (none) -> C8545
- R1, R2: value 5.1k -> (none); footprint Resistor_SMD:R_0805_2012Metric_Pad1.20x1.40mm_HandSolder -> (none); LCSC (none) -> C27834
- R3, R8: value 10k -> (none); footprint Resistor_SMD:R_0805_2012Metric_Pad1.20x1.40mm_HandSolder -> (none); LCSC (none) -> C17414
- R4, R5, R6, R7: value 100 -> (none); footprint Resistor_SMD:R_0805_2012Metric_Pad1.20x1.40mm_HandSolder -> (none); LCSC (none) -> C17408
- R9: value 1k -> (none); footprint Resistor_SMD:R_0805_2012Metric_Pad1.20x1.40mm_HandSolder -> (none); LCSC (none) -> C17513
- U1: value LM1117-3.3 -> (none); footprint Package_TO_SOT_SMD:SOT-223 -> (none); LCSC (none) -> C126027
- U2: value ESP32-WROOM-32D -> (none); footprint RF_Module:ESP32-WROOM-32 -> (none); LCSC (none) -> C473012
Connections:
- net +3V3: now also U3.6 (VDD), U3.7 (VREGIN)
- net +5V: now also U3.8 (VBUS)
- net D+: now also U3.4 (D+)
- net D-: now also U3.5 (D-)
- net GND: now also U3.29 (GND), U3.3 (GND)
- net RXD: now also U3.25 (RXD)
- net TXD: now also U3.26 (TXD)
- net at Q1.2 (S), R3.1: now also U3.24 (~{RTS})
- net at R9.2: now also U3.9 (~{RST})
- net at Q2.2 (S), R8.2: now also U3.28 (~{DTR})
- no-connect marks 22 -> 28
